Commit message: modified urdf files for checkpoint1 task1

File: my_rb1_description/urdf/my_rb1_robot.urdf (robot description, URDF)
Before this commit: robot visual, 16 links, 15 joints
Links:
- removed link box
- removed link gripper_pole
- removed link head
- removed link left_back_wheel
- removed link left_base
- removed link left_front_wheel
- removed link left_gripper
- removed link left_leg
- removed link left_tip
- removed link right_back_wheel
- removed link right_base
- removed link right_front_wheel
- removed link right_gripper
- removed link right_leg
- removed link right_tip
- added link back_caster; visual sphere radius=0.025
- added link front_caster; visual sphere radius=0.025
- added link front_laser; visual sphere radius=0.02
- added link left_wheel; visual cylinder length=0.03 radius=0.025
- added link right_wheel; visual cylinder length=0.03 radius=0.025
- link base_link: geometry visual cylinder length=0.3 radius=0.25
Joints:
- removed joint base_to_left_leg
- removed joint base_to_right_leg
- removed joint gripper_extension
- removed joint head_swivel
- removed joint left_back_wheel_joint
- removed joint left_base_joint
- removed joint left_front_wheel_joint
- removed joint left_gripper_joint
- removed joint left_tip_joint
- removed joint right_back_wheel_joint
- removed joint right_base_joint
- removed joint right_front_wheel_joint
- removed joint right_gripper_joint
- removed joint right_tip_joint
- removed joint tobox
- added joint joint_back_caster: type continuous, parent base_link, child back_caster, origin xyz=-0.1 0.0 -0.15 rpy=0.0 0.0 0.0, axis 1.0 1.0 0.0, limit lower=0.0 upper=0.0 effort=0.0 velocity=0.0
- added joint joint_front_caster: type continuous, parent base_link, child front_caster, origin xyz=0.1 0.0 -0.15 rpy=0.0 0.0 0.0, axis 1.0 1.0 0.0, limit lower=0.0 upper=0.0 effort=0.0 velocity=0.0
- added joint joint_front_laser: type continuous, parent base_link, child front_laser, origin xyz=0.25 0.0 0.12 rpy=0.0 0.0 0.0, axis 1.0 0.0 1.0, limit lower=0.0 upper=0.0 effort=0.0 velocity=0.0
- added joint joint_left_wheel: type fixed, parent base_link, child left_wheel, origin xyz=0.0 -0.25 -0.15 rpy=0.0 0.0 0.0
- added joint joint_right_wheel: type fixed, parent base_link, child right_wheel, origin xyz=0.0 0.25 -0.15 rpy=0.0 0.0 0.0

Commit message: add rviz to show tf and robot model

File: my_rb1_description/urdf/my_rb1_robot.urdf (robot description, URDF)
Before this commit: robot visual, 6 links, 5 joints
Joints:
- joint joint_left_wheel: axis (none) -> 0 1 0; limit (none) -> effort=10000 velocity=1000; type fixed -> continuous
- joint joint_right_wheel: axis (none) -> 0 1 0; limit (none) -> effort=10000 velocity=1000; type fixed -> continuous

Commit message: urdf for gazebo launch

File: my_rb1_description/urdf/my_rb1_robot.urdf (robot description, URDF)
Before this commit: robot visual, 6 links, 5 joints
Links:
- link back_caster: mass None -> 0.01; geometry collision sphere radius=0.025; visual sphere radius=0.025
- link base_link: mass None -> 1.0; geometry collision cylinder length=0.3 radius=0.25; visual cylinder length=0.3 radius=0.25
- link front_caster: mass None -> 0.01; geometry collision sphere radius=0.025; visual sphere radius=0.025
- link front_laser: mass None -> 0.01; geometry collision sphere radius=0.02; visual sphere radius=0.02
- link left_wheel: mass None -> 0.1; geometry collision cylinder length=0.03 radius=0.025; visual cylinder length=0.03 radius=0.025
- link right_wheel: mass None -> 0.1; geometry collision cylinder length=0.03 radius=0.025; visual cylinder length=0.03 radius=0.025

Commit message: final checkpoint source

File: my_rb1_description/urdf/my_rb1_robot.urdf (robot description, URDF)
Before this commit: robot my_rb1_robot, 6 links, 5 joints
Links:
- added link base_footprint, mass 0.0001; visual cylinder length=0.001 radius=0.001
- link back_caster: mass 0.01 -> 0.5
- link base_link: mass 1.0 -> 20.0
- link front_caster: mass 0.01 -> 0.5
- link left_wheel: mass 0.1 -> 2.0; geometry collision cylinder length=0.06 radius=0.05; visual cylinder length=0.06 radius=0.05
- link right_wheel: mass 0.1 -> 2.0; geometry collision cylinder length=0.06 radius=0.05; visual cylinder length=0.06 radius=0.05
Joints:
- added joint base_footprint_joint: type fixed, parent base_footprint, child base_link, origin xyz=0.0 0.0 0.12 rpy=0 0 0
- joint joint_back_caster: origin xyz=-0.1 0.0 -0.15 rpy=0.0 0.0 0.0 -> xyz=-0.15 0.0 -0.15 rpy=0.0 0.0 0.0
- joint joint_front_caster: origin xyz=0.1 0.0 -0.15 rpy=0.0 0.0 0.0 -> xyz=0.15 0.0 -0.15 rpy=0.0 0.0 0.0
- joint joint_front_laser: type continuous -> fixed
- joint joint_left_wheel: origin xyz=0.0 -0.25 -0.15 rpy=0.0 0.0 0.0 -> xyz=0.0 -0.225 -0.125 rpy=0.0 0.0 0.0
- joint joint_right_wheel: origin xyz=0.0 0.25 -0.15 rpy=0.0 0.0 0.0 -> xyz=0.0 0.225 -0.125 rpy=0.0 0.0 0.0

Commit message: fixed codes to revaluate checkpoint2

File: my_rb1_description/urdf/my_rb1_robot.urdf (robot description, URDF)
Before this commit: robot my_rb1_robot, 7 links, 6 joints
Joints:
- joint joint_left_wheel: origin xyz=0.0 -0.225 -0.125 rpy=0.0 0.0 0.0 -> xyz=0.0 0.225 -0.125 rpy=0.0 0.0 0.0
- joint joint_right_wheel: origin xyz=0.0 0.225 -0.125 rpy=0.0 0.0 0.0 -> xyz=0.0 -0.225 -0.125 rpy=0.0 0.0 0.0
